Commit message: fixed bugs of raytest, side, normal vector

File: urdf/painting/door.urdf (robot description, URDF)
Before this commit: robot carDoor, 1 links, 0 joints
Links:
- link carDoor_base_link: geometry collision mesh filename=test2.obj scale=1 1 1; visual mesh filename=test2.obj scale=1 1 1
